Commit message: Created new structure for URDF and OSIM.

File: Experiments/23links_human/templates/XSensModelStyle_URDFtemplate.urdf (robot description, URDF)
Before this commit: robot XSensStyleModel_template, 24 links, 23 joints
Links:
- removed link Ground
- link L3: geometry collision box size=L3_BOX_SIZE; visual box size=L3_BOX_SIZE
- link L5: geometry collision box size=L5_BOX_SIZE; visual box size=L5_BOX_SIZE
- link LeftFoot: mass FOOTMASS -> LEFTFOOTMASS; geometry collision box size=LEFTFOOT_BOX_SIZE; visual box size=LEFTFOOT_BOX_SIZE
- link LeftForeArm: mass FOREARMMASS -> LEFTFOREARMMASS; geometry collision cylinder length=LEFTFOREARMHEIGHT radius=LEFTFOREARMRADIUS; visual cylinder length=LEFTFOREARMHEIGHT radius=LEFTFOREARMRADIUS
- link LeftHand: mass HANDMASS -> LEFTHANDMASS; geometry collision box size=LEFTHAND_BOX_SIZE; visual box size=LEFTHAND_BOX_SIZE
- link LeftLowerLeg: mass LOWERLEGMASS -> LEFTLOWERLEGMASS; geometry collision cylinder length=LEFTLOWERLEGHEIGHT radius=LEFTLOWERLEGRADIUS; visual cylinder length=LEFTLOWERLEGHEIGHT radius=LEFTLOWERLEGRADIUS
- link LeftShoulder: mass SHOULDERMASS -> LEFTSHOULDERMASS; geometry collision cylinder length=LEFTSHOULDERHEIGHT radius=LEFTSHOULDERRADIUS; visual cylinder length=LEFTSHOULDERHEIGHT radius=LEFTSHOULDERRADIUS
- link LeftToe: mass TOEMASS -> LEFTTOEMASS; geometry collision box size=LEFTTOE_BOX_SIZE; visual box size=LEFTTOE_BOX_SIZE
- link LeftUpperArm: mass UPPERARMMASS -> LEFTUPPERARMMASS; geometry collision cylinder length=LEFTUPPERARMHEIGHT radius=LEFTUPPERARMRADIUS; visual cylinder length=LEFTUPPERARMHEIGHT radius=LEFTUPPERARMRADIUS
- link LeftUpperLeg: mass UPPERLEGMASS -> LEFTUPPERLEGMASS; geometry collision cylinder length=LEFTUPPERLEGHEIGHT radius=LEFTUPPERLEGRADIUS; visual cylinder length=LEFTUPPERLEGHEIGHT radius=LEFTUPPERLEGRADIUS
- link Pelvis: geometry collision box size=PELVIS_BOX_SIZE; visual box size=PELVIS_BOX_SIZE
- link RightFoot: mass FOOTMASS -> RIGHTFOOTMASS; geometry collision box size=RIGHTFOOT_BOX_SIZE; visual box size=RIGHTFOOT_BOX_SIZE
- link RightForeArm: mass FOREARMMASS -> RIGHTFOREARMMASS; geometry collision cylinder length=RIGHTFOREARMHEIGHT radius=RIGHTFOREARMRADIUS; visual cylinder length=RIGHTFOREARMHEIGHT radius=RIGHTFOREARMRADIUS
- link RightHand: mass HANDMASS -> RIGHTHANDMASS; geometry collision box size=RIGHTHAND_BOX_SIZE; visual box size=RIGHTHAND_BOX_SIZE
- link RightLowerLeg: mass LOWERLEGMASS -> RIGHTLOWERLEGMASS; geometry collision cylinder length=RIGHTLOWERLEGHEIGHT radius=RIGHTLOWERLEGRADIUS; visual cylinder length=RIGHTLOWERLEGHEIGHT radius=RIGHTLOWERLEGRADIUS
- link RightShoulder: mass SHOULDERMASS -> RIGHTSHOULDERMASS; geometry collision cylinder length=RIGHTSHOULDERHEIGHT radius=RIGHTSHOULDERRADIUS; visual cylinder length=RIGHTSHOULDERHEIGHT radius=RIGHTSHOULDERRADIUS
- link RightToe: mass TOEMASS -> RIGHTTOEMASS; geometry collision box size=RIGHTTOE_BOX_SIZE; visual box size=RIGHTTOE_BOX_SIZE
- link RightUpperArm: mass UPPERARMMASS -> RIGHTUPPERARMMASS; geometry collision cylinder length=RIGHTUPPERARMHEIGHT radius=RIGHTUPPERARMRADIUS; visual cylinder length=RIGHTUPPERARMHEIGHT radius=RIGHTUPPERARMRADIUS
- link RightUpperLeg: mass UPPERLEGMASS -> RIGHTUPPERLEGMASS; geometry collision cylinder length=RIGHTUPPERLEGHEIGHT radius=RIGHTUPPERLEGRADIUS; visual cylinder length=RIGHTUPPERLEGHEIGHT radius=RIGHTUPPERLEGRADIUS
- link T12: geometry collision box size=T12_BOX_SIZE; visual box size=T12_BOX_SIZE
- link T8: geometry collision box size=T8_BOX_SIZE; visual box size=T8_BOX_SIZE
Joints:
- removed joint jGround_LeftFoot
- joint jC1Head: origin xyz=0 0 NECKHEIGHT rpy=0 0 0 -> xyz=jC1Head_ORIGIN rpy=0 0 0
- joint jL1T12: origin xyz=0 0 L3HEIGHT rpy=0 0 0 -> xyz=jL1T12_ORIGIN rpy=0 0 0
- joint jL4L3: origin xyz=0 0 L5HEIGHT rpy=0 0 0 -> xyz=jL4L3_ORIGIN rpy=0 0 0
- joint jL5S1: origin xyz=0 -HIPPOSY PELVISBETA rpy=0 0 0 -> xyz=jL5S1_ORIGIN rpy=0 0 0
- joint jLeftAnkle: child LeftLowerLeg -> LeftFoot; origin xyz=-ANKLEPOSX 0 FOOTBETA rpy=0 0 0 -> xyz=jLeftAnkle_ORIGIN rpy=0 0 0; parent LeftFoot -> LeftLowerLeg
- joint jLeftBallFoot: origin xyz=FOOTHALFGAMMA 0 FOOTHALFBETA rpy=0 0 0 -> xyz=jLeftBallFoot_ORIGIN rpy=0 0 0
- joint jLeftC7Shoulder: origin xyz=0 T8HALFALFA SHOULDERURDFPOSZ rpy=0 0 0 -> xyz=jLeftC7Shoulder_ORIGIN rpy=0 0 0
- joint jLeftElbow: origin xyz=0 UPPERARMRADIUS -ARMURDFPOSZ rpy=0 0 0 -> xyz=jLeftElbow_ORIGIN rpy=0 0 0
- joint jLeftHip: child Pelvis -> LeftUpperLeg; origin xyz=0 0 UPPERLEGHEIGHT rpy=0 0 0 -> xyz=jLeftHip_ORIGIN rpy=0 0 0; parent LeftUpperLeg -> Pelvis
- joint jLeftKnee: child LeftUpperLeg -> LeftLowerLeg; origin xyz=0 0 LOWERLEGHEIGHT rpy=0 0 0 -> xyz=jLeftKnee_ORIGIN rpy=0 0 0; parent LeftLowerLeg -> LeftUpperLeg
- joint jLeftShoulder: origin xyz=0 SHOULDERHEIGHT 0 rpy=0 0 0 -> xyz=jLeftShoulder_ORIGIN rpy=0 0 0
- joint jLeftWrist: origin xyz=0 0 -FOREARMHEIGHT rpy=0 0 0 -> xyz=jLeftWrist_ORIGIN rpy=0 0 0
- joint jRightAnkle: origin xyz=0 0 -LOWERLEGHEIGHT rpy=0 0 0 -> xyz=jRightAnkle_ORIGIN rpy=0 0 0
- joint jRightBallFoot: origin xyz=TOEPOSX 0 -FOOTHALFBETA rpy=0 0 0 -> xyz=jRightBallFoot_ORIGIN rpy=0 0 0
- joint jRightC7Shoulder: origin xyz=0 -T8HALFALFA SHOULDERURDFPOSZ rpy=0 0 0 -> xyz=jRightC7Shoulder_ORIGIN rpy=0 0 0
- joint jRightElbow: origin xyz=0 -UPPERARMRADIUS -ARMURDFPOSZ rpy=0 0 0 -> xyz=jRightElbow_ORIGIN rpy=0 0 0
- joint jRightHip: origin xyz=0 -HIPDOUBLEPOSY 0 rpy=0 0 0 -> xyz=jRightHip_ORIGIN rpy=0 0 0
- joint jRightKnee: origin xyz=0 0 -UPPERLEGHEIGHT rpy=0 0 0 -> xyz=jRightKnee_ORIGIN rpy=0 0 0
- joint jRightShoulder: origin xyz=0 -SHOULDERHEIGHT 0 rpy=0 0 0 -> xyz=jRightShoulder_ORIGIN rpy=0 0 0
- joint jRightWrist: origin xyz=0 0 -FOREARMHEIGHT rpy=0 0 0 -> xyz=jRightWrist_ORIGIN rpy=0 0 0
- joint jT1C7: origin xyz=0 0 T8BETA rpy=0 0 0 -> xyz=jT1C7_ORIGIN rpy=0 0 0
- joint jT9T8: origin xyz=0 0 T12HEIGHT rpy=0 0 0 -> xyz=jT9T8_ORIGIN rpy=0 0 0
