Commit message: URDFtemplate joints as combination of 3 rotational
All joints as combination of 3 rotational joints

File: Experiments/23links_human/templates/XSensModelStyle_URDFtemplate.urdf (robot description, URDF)
Before this commit: robot XSensStyleModel_template, 23 links, 22 joints
Links:
- added link Head_f1, mass FAKEMASS; collision box size=FAKEDIM FAKEDIM FAKEDIM; visual box size=FAKEDIM FAKEDIM FAKEDIM
- added link Head_f2, mass FAKEMASS; collision box size=FAKEDIM FAKEDIM FAKEDIM; visual box size=FAKEDIM FAKEDIM FAKEDIM
- added link L3_f1, mass FAKEMASS; collision box size=FAKEDIM FAKEDIM FAKEDIM; visual box size=FAKEDIM FAKEDIM FAKEDIM
- added link L3_f2, mass FAKEMASS; collision box size=FAKEDIM FAKEDIM FAKEDIM; visual box size=FAKEDIM FAKEDIM FAKEDIM
- added link L5_f1, mass FAKEMASS; collision box size=FAKEDIM FAKEDIM FAKEDIM; visual box size=FAKEDIM FAKEDIM FAKEDIM
- added link L5_f2, mass FAKEMASS; collision box size=FAKEDIM FAKEDIM FAKEDIM; visual box size=FAKEDIM FAKEDIM FAKEDIM
- added link LeftFoot_f1, mass FAKEMASS; collision box size=FAKEDIM FAKEDIM FAKEDIM; visual box size=FAKEDIM FAKEDIM FAKEDIM
- added link LeftFoot_f2, mass FAKEMASS; collision box size=FAKEDIM FAKEDIM FAKEDIM; visual box size=FAKEDIM FAKEDIM FAKEDIM
- added link LeftForeArm_f1, mass FAKEMASS; collision box size=FAKEDIM FAKEDIM FAKEDIM; visual box size=FAKEDIM FAKEDIM FAKEDIM
- added link LeftForeArm_f2, mass FAKEMASS; collision box size=FAKEDIM FAKEDIM FAKEDIM; visual box size=FAKEDIM FAKEDIM FAKEDIM
- added link LeftHand_f1, mass FAKEMASS; collision box size=FAKEDIM FAKEDIM FAKEDIM; visual box size=FAKEDIM FAKEDIM FAKEDIM
- added link LeftHand_f2, mass FAKEMASS; collision box size=FAKEDIM FAKEDIM FAKEDIM; visual box size=FAKEDIM FAKEDIM FAKEDIM
- added link LeftLowerLeg_f1, mass FAKEMASS; collision box size=FAKEDIM FAKEDIM FAKEDIM; visual box size=FAKEDIM FAKEDIM FAKEDIM
- added link LeftLowerLeg_f2, mass FAKEMASS; collision box size=FAKEDIM FAKEDIM FAKEDIM; visual box size=FAKEDIM FAKEDIM FAKEDIM
- added link LeftShoulder_f1, mass FAKEMASS; collision box size=FAKEDIM FAKEDIM FAKEDIM; visual box size=FAKEDIM FAKEDIM FAKEDIM
- added link LeftShoulder_f2, mass FAKEMASS; collision box size=FAKEDIM FAKEDIM FAKEDIM; visual box size=FAKEDIM FAKEDIM FAKEDIM
- added link LeftToe_f1, mass FAKEMASS; collision box size=FAKEDIM FAKEDIM FAKEDIM; visual box size=FAKEDIM FAKEDIM FAKEDIM
- added link LeftToe_f2, mass FAKEMASS; collision box size=FAKEDIM FAKEDIM FAKEDIM; visual box size=FAKEDIM FAKEDIM FAKEDIM
- added link LeftUpperArm_f1, mass FAKEMASS; collision box size=FAKEDIM FAKEDIM FAKEDIM; visual box size=FAKEDIM FAKEDIM FAKEDIM
- added link LeftUpperArm_f2, mass FAKEMASS; collision box size=FAKEDIM FAKEDIM FAKEDIM; visual box size=FAKEDIM FAKEDIM FAKEDIM
- added link LeftUpperLeg_f1, mass FAKEMASS; collision box size=FAKEDIM FAKEDIM FAKEDIM; visual box size=FAKEDIM FAKEDIM FAKEDIM
- added link LeftUpperLeg_f2, mass FAKEMASS; collision box size=FAKEDIM FAKEDIM FAKEDIM; visual box size=FAKEDIM FAKEDIM FAKEDIM
- added link Neck_f1, mass FAKEMASS; collision box size=FAKEDIM FAKEDIM FAKEDIM; visual box size=FAKEDIM FAKEDIM FAKEDIM
- added link Neck_f2, mass FAKEMASS; collision box size=FAKEDIM FAKEDIM FAKEDIM; visual box size=FAKEDIM FAKEDIM FAKEDIM
- added link RightFoot_f1, mass FAKEMASS; collision box size=FAKEDIM FAKEDIM FAKEDIM; visual box size=FAKEDIM FAKEDIM FAKEDIM
- added link RightFoot_f2, mass FAKEMASS; collision box size=FAKEDIM FAKEDIM FAKEDIM; visual box size=FAKEDIM FAKEDIM FAKEDIM
- added link RightForeArm_f1, mass FAKEMASS; collision box size=FAKEDIM FAKEDIM FAKEDIM; visual box size=FAKEDIM FAKEDIM FAKEDIM
- added link RightForeArm_f2, mass FAKEMASS; collision box size=FAKEDIM FAKEDIM FAKEDIM; visual box size=FAKEDIM FAKEDIM FAKEDIM
- added link RightHand_f1, mass FAKEMASS; collision box size=FAKEDIM FAKEDIM FAKEDIM; visual box size=FAKEDIM FAKEDIM FAKEDIM
- added link RightHand_f2, mass FAKEMASS; collision box size=FAKEDIM FAKEDIM FAKEDIM; visual box size=FAKEDIM FAKEDIM FAKEDIM
- added link RightLowerLeg_f1, mass FAKEMASS; collision box size=FAKEDIM FAKEDIM FAKEDIM; visual box size=FAKEDIM FAKEDIM FAKEDIM
- added link RightLowerLeg_f2, mass FAKEMASS; collision box size=FAKEDIM FAKEDIM FAKEDIM; visual box size=FAKEDIM FAKEDIM FAKEDIM
- added link RightShoulder_f1, mass FAKEMASS; collision box size=FAKEDIM FAKEDIM FAKEDIM; visual box size=FAKEDIM FAKEDIM FAKEDIM
- added link RightShoulder_f2, mass FAKEMASS; collision box size=FAKEDIM FAKEDIM FAKEDIM; visual box size=FAKEDIM FAKEDIM FAKEDIM
- added link RightToe_f1, mass FAKEMASS; collision box size=FAKEDIM FAKEDIM FAKEDIM; visual box size=FAKEDIM FAKEDIM FAKEDIM
- added link RightToe_f2, mass FAKEMASS; collision box size=FAKEDIM FAKEDIM FAKEDIM; visual box size=FAKEDIM FAKEDIM FAKEDIM
- added link RightUpperArm_f1, mass FAKEMASS; collision box size=FAKEDIM FAKEDIM FAKEDIM; visual box size=FAKEDIM FAKEDIM FAKEDIM
- added link RightUpperArm_f2, mass FAKEMASS; collision box size=FAKEDIM FAKEDIM FAKEDIM; visual box size=FAKEDIM FAKEDIM FAKEDIM
- added link RightUpperLeg_f1, mass FAKEMASS; collision box size=FAKEDIM FAKEDIM FAKEDIM; visual box size=FAKEDIM FAKEDIM FAKEDIM
- added link RightUpperLeg_f2, mass FAKEMASS; collision box size=FAKEDIM FAKEDIM FAKEDIM; visual box size=FAKEDIM FAKEDIM FAKEDIM
- added link T12_f1, mass FAKEMASS; collision box size=FAKEDIM FAKEDIM FAKEDIM; visual box size=FAKEDIM FAKEDIM FAKEDIM
- added link T12_f2, mass FAKEMASS; collision box size=FAKEDIM FAKEDIM FAKEDIM; visual box size=FAKEDIM FAKEDIM FAKEDIM
- added link T8_f1, mass FAKEMASS; collision box size=FAKEDIM FAKEDIM FAKEDIM; visual box size=FAKEDIM FAKEDIM FAKEDIM
- added link T8_f2, mass FAKEMASS; collision box size=FAKEDIM FAKEDIM FAKEDIM; visual box size=FAKEDIM FAKEDIM FAKEDIM
Joints:
- removed joint jC1Head
- removed joint jL1T12
- removed joint jL4L3
- removed joint jL5S1
- removed joint jLeftAnkle
- removed joint jLeftBallFoot
- removed joint jLeftC7Shoulder
- removed joint jLeftElbow
- removed joint jLeftHip
- removed joint jLeftKnee
- removed joint jLeftShoulder
- removed joint jLeftWrist
- removed joint jRightAnkle
- removed joint jRightBallFoot
- removed joint jRightC7Shoulder
- removed joint jRightElbow
- removed joint jRightHip
- removed joint jRightKnee
- removed joint jRightShoulder
- removed joint jRightWrist
- removed joint jT1C7
- removed joint jT9T8
- added joint jC1Head_rotx: type revolute, parent Neck, child Head_f1, origin xyz=jC1Head_ORIGIN rpy=0 0 0, axis 1 0 0, limit lower=-10.0 effort=30 velocity=1.0
- added joint jC1Head_roty: type revolute, parent Head_f1, child Head_f2, origin xyz=0 0 0 rpy=0 0 0, axis 0 1 0, limit lower=-10.0 effort=30 velocity=1.0
- added joint jC1Head_rotz: type revolute, parent Head_f2, child Head, origin xyz=0 0 0 rpy=0 0 0, axis 0 0 1, limit lower=-10.0 effort=30 velocity=1.0
- added joint jL1T12_rotx: type revolute, parent L3, child T12_f1, origin xyz=jL1T12_ORIGIN rpy=0 0 0, axis 1 0 0, limit lower=-10.0 effort=30 velocity=1.0
- added joint jL1T12_roty: type revolute, parent T12_f1, child T12_f2, origin xyz=0 0 0 rpy=0 0 0, axis 0 1 0, limit lower=-10.0 effort=30 velocity=1.0
- added joint jL1T12_rotz: type revolute, parent T12_f2, child T12, origin xyz=0 0 0 rpy=0 0 0, axis 0 0 1, limit lower=-10.0 effort=30 velocity=1.0
- added joint jL4L3_rotx: type revolute, parent L5, child L3_f1, origin xyz=jL4L3_ORIGIN rpy=0 0 0, axis 1 0 0, limit lower=-10.0 effort=30 velocity=1.0
- added joint jL4L3_roty: type revolute, parent L3_f1, child L3_f2, origin xyz=0 0 0 rpy=0 0 0, axis 0 1 0, limit lower=-10.0 effort=30 velocity=1.0
- added joint jL4L3_rotz: type revolute, parent L3_f2, child L3, origin xyz=0 0 0 rpy=0 0 0, axis 0 0 1, limit lower=-10.0 effort=30 velocity=1.0
- added joint jL5S1_rotx: type revolute, parent Pelvis, child L5_f1, origin xyz=jL5S1_ORIGIN rpy=0 0 0, axis 1 0 0, limit lower=-10.0 effort=30 velocity=1.0
- added joint jL5S1_roty: type revolute, parent L5_f1, child L5_f2, origin xyz=0 0 0 rpy=0 0 0, axis 0 1 0, limit lower=-10.0 effort=30 velocity=1.0
- added joint jL5S1_rotz: type revolute, parent L5_f2, child L5, origin xyz=0 0 0 rpy=0 0 0, axis 0 0 1, limit lower=-10.0 effort=30 velocity=1.0
- added joint jLeftAnkle_rotx: type revolute, parent LeftLowerLeg, child LeftFoot_f1, origin xyz=jLeftAnkle_ORIGIN rpy=0 0 0, axis 1 0 0, limit lower=-10.0 effort=30 velocity=1.0
- added joint jLeftAnkle_roty: type revolute, parent LeftFoot_f1, child LeftFoot_f2, origin xyz=0 0 0 rpy=0 0 0, axis 0 1 0, limit lower=-10.0 effort=30 velocity=1.0
- added joint jLeftAnkle_rotz: type revolute, parent LeftFoot_f2, child LeftFoot, origin xyz=0 0 0 rpy=0 0 0, axis 0 0 1, limit lower=-10.0 effort=30 velocity=1.0
- added joint jLeftBallFoot_rotx: type revolute, parent LeftFoot, child LeftToe_f1, origin xyz=jLeftBallFoot_ORIGIN rpy=0 0 0, axis 1 0 0, limit lower=-10.0 effort=30 velocity=1.0
- added joint jLeftBallFoot_roty: type revolute, parent LeftToe_f1, child LeftToe_f2, origin xyz=0 0 0 rpy=0 0 0, axis 0 1 0, limit lower=-10.0 effort=30 velocity=1.0
- added joint jLeftBallFoot_rotz: type revolute, parent LeftToe_f2, child LeftToe, origin xyz=0 0 0 rpy=0 0 0, axis 0 0 1, limit lower=-10.0 effort=30 velocity=1.0
- added joint jLeftC7Shoulder_rotx: type revolute, parent T8, child LeftShoulder_f1, origin xyz=jLeftC7Shoulder_ORIGIN rpy=0 0 0, axis 1 0 0, limit lower=-10.0 effort=30 velocity=1.0
- added joint jLeftC7Shoulder_roty: type revolute, parent LeftShoulder_f1, child LeftShoulder_f2, origin xyz=0 0 0 rpy=0 0 0, axis 0 1 0, limit lower=-10.0 effort=30 velocity=1.0
- added joint jLeftC7Shoulder_rotz: type revolute, parent LeftShoulder_f2, child LeftShoulder, origin xyz=0 0 0 rpy=0 0 0, axis 0 0 1, limit lower=-10.0 effort=30 velocity=1.0
- added joint jLeftElbow_rotx: type revolute, parent LeftUpperArm, child LeftForeArm_f1, origin xyz=jLeftElbow_ORIGIN rpy=0 0 0, axis 1 0 0, limit lower=-10.0 effort=30 velocity=1.0
- added joint jLeftElbow_roty: type revolute, parent LeftForeArm_f1, child LeftForeArm_f2, origin xyz=0 0 0 rpy=0 0 0, axis 0 1 0, limit lower=-10.0 effort=30 velocity=1.0
- added joint jLeftElbow_rotz: type revolute, parent LeftForeArm_f2, child LeftForeArm, origin xyz=0 0 0 rpy=0 0 0, axis 0 0 1, limit lower=-10.0 effort=30 velocity=1.0
- added joint jLeftHip_rotx: type revolute, parent Pelvis, child LeftUpperLeg_f1, origin xyz=jLeftHip_ORIGIN rpy=0 0 0, axis 1 0 0, limit lower=-10.0 effort=30 velocity=1.0
- added joint jLeftHip_roty: type revolute, parent LeftUpperLeg_f1, child LeftUpperLeg_f2, origin xyz=0 0 0 rpy=0 0 0, axis 0 1 0, limit lower=-10.0 effort=30 velocity=1.0
- added joint jLeftHip_rotz: type revolute, parent LeftUpperLeg_f2, child LeftUpperLeg, origin xyz=0 0 0 rpy=0 0 0, axis 0 0 1, limit lower=-10.0 effort=30 velocity=1.0
- added joint jLeftKnee_rotx: type revolute, parent LeftUpperLeg, child LeftLowerLeg_f1, origin xyz=jLeftKnee_ORIGIN rpy=0 0 0, axis 1 0 0, limit lower=-10.0 effort=30 velocity=1.0
- added joint jLeftKnee_roty: type revolute, parent LeftLowerLeg_f1, child LeftLowerLeg_f2, origin xyz=0 0 0 rpy=0 0 0, axis 0 1 0, limit lower=-10.0 effort=30 velocity=1.0
- added joint jLeftKnee_rotz: type revolute, parent LeftLowerLeg_f2, child LeftLowerLeg, origin xyz=0 0 0 rpy=0 0 0, axis 0 0 1, limit lower=-10.0 effort=30 velocity=1.0
- added joint jLeftShoulder_rotx: type revolute, parent LeftShoulder, child LeftUpperArm_f1, origin xyz=jLeftShoulder_ORIGIN rpy=0 0 0, axis 1 0 0, limit lower=-10.0 upper=10.0 effort=30 velocity=1.0
- added joint jLeftShoulder_roty: type revolute, parent LeftUpperArm_f1, child LeftUpperArm_f2, origin xyz=0 0 0 rpy=0 0 0, axis 0 1 0, limit lower=-10.0 upper=10.0 effort=30 velocity=1.0
- added joint jLeftShoulder_rotz: type revolute, parent LeftUpperArm_f2, child LeftUpperArm, origin xyz=0 0 0 rpy=0 0 0, axis 0 0 1, limit lower=-10.0 upper=10.0 effort=30 velocity=1.0
- added joint jLeftWrist_rotx: type revolute, parent LeftForeArm, child LeftHand_f1, origin xyz=jLeftWrist_ORIGIN rpy=0 0 0, axis 1 0 0, limit lower=-10.0 effort=30 velocity=1.0
- added joint jLeftWrist_roty: type revolute, parent LeftHand_f1, child LeftHand_f2, origin xyz=0 0 0 rpy=0 0 0, axis 0 1 0, limit lower=-10.0 effort=30 velocity=1.0
- added joint jLeftWrist_rotz: type revolute, parent LeftHand_f2, child LeftHand, origin xyz=0 0 0 rpy=0 0 0, axis 0 0 1, limit lower=-10.0 effort=30 velocity=1.0
- added joint jRightAnkle_rotx: type revolute, parent RightLowerLeg, child RightFoot_f1, origin xyz=jRightAnkle_ORIGIN rpy=0 0 0, axis 1 0 0, limit lower=-10.0 effort=30 velocity=1.0
- added joint jRightAnkle_roty: type revolute, parent RightFoot_f1, child RightFoot_f2, origin xyz=0 0 0 rpy=0 0 0, axis 0 1 0, limit lower=-10.0 effort=30 velocity=1.0
- added joint jRightAnkle_rotz: type revolute, parent RightFoot_f2, child RightFoot, origin xyz=0 0 0 rpy=0 0 0, axis 0 0 1, limit lower=-10.0 effort=30 velocity=1.0
- added joint jRightBallFoot_rotx: type revolute, parent RightFoot, child RightToe_f1, origin xyz=jRightBallFoot_ORIGIN rpy=0 0 0, axis 1 0 0, limit lower=-10.0 effort=30 velocity=1.0
- added joint jRightBallFoot_roty: type revolute, parent RightToe_f1, child RightToe_f2, origin xyz=0 0 0 rpy=0 0 0, axis 0 1 0, limit lower=-10.0 effort=30 velocity=1.0
- added joint jRightBallFoot_rotz: type revolute, parent RightToe_f2, child RightToe, origin xyz=0 0 0 rpy=0 0 0, axis 0 0 1, limit lower=-10.0 effort=30 velocity=1.0
- added joint jRightC7Shoulder_rotx: type revolute, parent T8, child RightShoulder_f1, origin xyz=jRightC7Shoulder_ORIGIN rpy=0 0 0, axis 1 0 0, limit lower=-10.0 effort=30 velocity=1.0
- added joint jRightC7Shoulder_roty: type revolute, parent RightShoulder_f1, child RightShoulder_f2, origin xyz=0 0 0 rpy=0 0 0, axis 0 1 0, limit lower=-10.0 effort=30 velocity=1.0
- added joint jRightC7Shoulder_rotz: type revolute, parent RightShoulder_f2, child RightShoulder, origin xyz=0 0 0 rpy=0 0 0, axis 0 0 1, limit lower=-10.0 effort=30 velocity=1.0
- added joint jRightElbow_rotx: type revolute, parent RightUpperArm, child RightForeArm_f1, origin xyz=jRightElbow_ORIGIN rpy=0 0 0, axis 1 0 0, limit lower=-10.0 effort=30 velocity=1.0
- added joint jRightElbow_roty: type revolute, parent RightForeArm_f1, child RightForeArm_f2, origin xyz=0 0 0 rpy=0 0 0, axis 0 1 0, limit lower=-10.0 effort=30 velocity=1.0
- added joint jRightElbow_rotz: type revolute, parent RightForeArm_f2, child RightForeArm, origin xyz=0 0 0 rpy=0 0 0, axis 0 0 1, limit lower=-10.0 effort=30 velocity=1.0
- added joint jRightHip_rotx: type revolute, parent Pelvis, child RightUpperLeg_f1, origin xyz=jRightHip_ORIGIN rpy=0 0 0, axis 1 0 0, limit lower=-10.0 effort=30 velocity=1.0
- added joint jRightHip_roty: type revolute, parent RightUpperLeg_f1, child RightUpperLeg_f2, origin xyz=0 0 0 rpy=0 0 0, axis 0 1 0, limit lower=-10.0 effort=30 velocity=1.0
- added joint jRightHip_rotz: type revolute, parent RightUpperLeg_f2, child RightUpperLeg, origin xyz=0 0 0 rpy=0 0 0, axis 0 0 1, limit lower=-10.0 effort=30 velocity=1.0
- added joint jRightKnee_rotx: type revolute, parent RightUpperLeg, child RightLowerLeg_f1, origin xyz=jRightKnee_ORIGIN rpy=0 0 0, axis 1 0 0, limit lower=-10.0 effort=30 velocity=1.0
- added joint jRightKnee_roty: type revolute, parent RightLowerLeg_f1, child RightLowerLeg_f2, origin xyz=0 0 0 rpy=0 0 0, axis 0 1 0, limit lower=-10.0 effort=30 velocity=1.0
- added joint jRightKnee_rotz: type revolute, parent RightLowerLeg_f2, child RightLowerLeg, origin xyz=0 0 0 rpy=0 0 0, axis 0 0 1, limit lower=-10.0 effort=30 velocity=1.0
- added joint jRightShoulder_rotx: type revolute, parent RightShoulder, child RightUpperArm_f1, origin xyz=jRightShoulder_ORIGIN rpy=0 0 0, axis 1 0 0, limit lower=-10.0 upper=10.0 effort=30 velocity=1.0
- added joint jRightShoulder_roty: type revolute, parent RightUpperArm_f1, child RightUpperArm_f2, origin xyz=0 0 0 rpy=0 0 0, axis 0 1 0, limit lower=-10.0 upper=10.0 effort=30 velocity=1.0
- added joint jRightShoulder_rotz: type revolute, parent RightUpperArm_f2, child RightUpperArm, origin xyz=0 0 0 rpy=0 0 0, axis 0 0 1, limit lower=-10.0 upper=10.0 effort=30 velocity=1.0
- added joint jRightWrist_rotx: type revolute, parent RightForeArm, child RightHand_f1, origin xyz=jRightWrist_ORIGIN rpy=0 0 0, axis 1 0 0, limit lower=-10.0 effort=30 velocity=1.0
- added joint jRightWrist_roty: type revolute, parent RightHand_f1, child RightHand_f2, origin xyz=0 0 0 rpy=0 0 0, axis 0 1 0, limit lower=-10.0 effort=30 velocity=1.0
- added joint jRightWrist_rotz: type revolute, parent RightHand_f2, child RightHand, origin xyz=0 0 0 rpy=0 0 0, axis 0 0 1, limit lower=-10.0 effort=30 velocity=1.0
- added joint jT1C7_rotx: type revolute, parent T8, child Neck_f1, origin xyz=jT1C7_ORIGIN rpy=0 0 0, axis 1 0 0, limit lower=-10.0 effort=30 velocity=1.0
- added joint jT1C7_roty: type revolute, parent Neck_f1, child Neck_f2, origin xyz=0 0 0 rpy=0 0 0, axis 0 1 0, limit lower=-10.0 effort=30 velocity=1.0
- added joint jT1C7_rotz: type revolute, parent Neck_f2, child Neck, origin xyz=0 0 0 rpy=0 0 0, axis 0 0 1, limit lower=-10.0 effort=30 velocity=1.0
- added joint jT9T8_rotx: type revolute, parent T12, child T8_f1, origin xyz=jT9T8_ORIGIN rpy=0 0 0, axis 1 0 0, limit lower=-10.0 effort=30 velocity=1.0
- added joint jT9T8_roty: type revolute, parent T8_f1, child T8_f2, origin xyz=0 0 0 rpy=0 0 0, axis 0 1 0, limit lower=-10.0 effort=30 velocity=1.0
- added joint jT9T8_rotz: type revolute, parent T8_f2, child T8, origin xyz=0 0 0 rpy=0 0 0, axis 0 0 1, limit lower=-10.0 effort=30 velocity=1.0

Commit message: Update XSensModelStyle_URDFtemplate.urdf

File: Experiments/23links_human/templates/XSensModelStyle_URDFtemplate.urdf (robot description, URDF)
Before this commit: robot XSensStyleModel_template, 67 links, 66 joints
Links:
- link Head_f1: mass FAKEMASS -> 0 0 0; geometry collision box size=0 0 0; visual box size=0 0 0
- link Head_f2: mass FAKEMASS -> 0 0 0; geometry collision box size=0 0 0; visual box size=0 0 0
- link L3_f1: mass FAKEMASS -> 0 0 0; geometry collision box size=0 0 0; visual box size=0 0 0
- link L3_f2: mass FAKEMASS -> 0 0 0; geometry collision box size=0 0 0; visual box size=0 0 0
- link L5_f1: mass FAKEMASS -> 0 0 0; geometry collision box size=0 0 0; visual box size=0 0 0
- link L5_f2: mass FAKEMASS -> 0 0 0; geometry collision box size=0 0 0; visual box size=0 0 0
- link LeftFoot_f1: mass FAKEMASS -> 0 0 0; geometry collision box size=0 0 0; visual box size=0 0 0
- link LeftFoot_f2: mass FAKEMASS -> 0 0 0; geometry collision box size=0 0 0; visual box size=0 0 0
- link LeftForeArm_f1: mass FAKEMASS -> 0 0 0; geometry collision box size=0 0 0; visual box size=0 0 0
- link LeftForeArm_f2: mass FAKEMASS -> 0 0 0; geometry collision box size=0 0 0; visual box size=0 0 0
- link LeftHand_f1: mass FAKEMASS -> 0 0 0; geometry collision box size=0 0 0; visual box size=0 0 0
- link LeftHand_f2: mass FAKEMASS -> 0 0 0; geometry collision box size=0 0 0; visual box size=0 0 0
- link LeftLowerLeg_f1: mass FAKEMASS -> 0 0 0; geometry collision box size=0 0 0; visual box size=0 0 0
- link LeftLowerLeg_f2: mass FAKEMASS -> 0 0 0; geometry collision box size=0 0 0; visual box size=0 0 0
- link LeftShoulder_f1: mass FAKEMASS -> 0 0 0; geometry collision box size=0 0 0; visual box size=0 0 0
- link LeftShoulder_f2: mass FAKEMASS -> 0 0 0; geometry collision box size=0 0 0; visual box size=0 0 0
- link LeftToe_f1: mass FAKEMASS -> 0 0 0; geometry collision box size=0 0 0; visual box size=0 0 0
- link LeftToe_f2: mass FAKEMASS -> 0 0 0; geometry collision box size=0 0 0; visual box size=0 0 0
- link LeftUpperArm_f1: mass FAKEMASS -> 0 0 0; geometry collision box size=0 0 0; visual box size=0 0 0
- link LeftUpperArm_f2: mass FAKEMASS -> 0 0 0; geometry collision box size=0 0 0; visual box size=0 0 0
- link LeftUpperLeg_f1: mass FAKEMASS -> 0 0 0; geometry collision box size=0 0 0; visual box size=0 0 0
- link LeftUpperLeg_f2: mass FAKEMASS -> 0 0 0; geometry collision box size=0 0 0; visual box size=0 0 0
- link Neck_f1: mass FAKEMASS -> 0 0 0; geometry collision box size=0 0 0; visual box size=0 0 0
- link Neck_f2: mass FAKEMASS -> 0 0 0; geometry collision box size=0 0 0; visual box size=0 0 0
- link RightFoot_f1: mass FAKEMASS -> 0 0 0; geometry collision box size=0 0 0; visual box size=0 0 0
- link RightFoot_f2: mass FAKEMASS -> 0 0 0; geometry collision box size=0 0 0; visual box size=0 0 0
- link RightForeArm_f1: mass FAKEMASS -> 0 0 0; geometry collision box size=0 0 0; visual box size=0 0 0
- link RightForeArm_f2: mass FAKEMASS -> 0 0 0; geometry collision box size=0 0 0; visual box size=0 0 0
- link RightHand_f1: mass FAKEMASS -> 0 0 0; geometry collision box size=0 0 0; visual box size=0 0 0
- link RightHand_f2: mass FAKEMASS -> 0 0 0; geometry collision box size=0 0 0; visual box size=0 0 0
- link RightLowerLeg_f1: mass FAKEMASS -> 0 0 0; geometry collision box size=0 0 0; visual box size=0 0 0
- link RightLowerLeg_f2: mass FAKEMASS -> 0 0 0; geometry collision box size=0 0 0; visual box size=0 0 0
- link RightShoulder_f1: mass FAKEMASS -> 0 0 0; geometry collision box size=0 0 0; visual box size=0 0 0
- link RightShoulder_f2: mass FAKEMASS -> 0 0 0; geometry collision box size=0 0 0; visual box size=0 0 0
- link RightToe_f1: mass FAKEMASS -> 0 0 0; geometry collision box size=0 0 0; visual box size=0 0 0
- link RightToe_f2: mass FAKEMASS -> 0 0 0; geometry collision box size=0 0 0; visual box size=0 0 0
- link RightUpperArm_f1: mass FAKEMASS -> 0 0 0; geometry collision box size=0 0 0; visual box size=0 0 0
- link RightUpperArm_f2: mass FAKEMASS -> 0 0 0; geometry collision box size=0 0 0; visual box size=0 0 0
- link RightUpperLeg_f1: mass FAKEMASS -> 0 0 0; geometry collision box size=0 0 0; visual box size=0 0 0
- link RightUpperLeg_f2: mass FAKEMASS -> 0 0 0; geometry collision box size=0 0 0; visual box size=0 0 0
- link T12_f1: mass FAKEMASS -> 0 0 0; geometry collision box size=0 0 0; visual box size=0 0 0
- link T12_f2: mass FAKEMASS -> 0 0 0; geometry collision box size=0 0 0; visual box size=0 0 0
- link T8_f1: mass FAKEMASS -> 0 0 0; geometry collision box size=0 0 0; visual box size=0 0 0
- link T8_f2: mass FAKEMASS -> 0 0 0; geometry collision box size=0 0 0; visual box size=0 0 0
