Commit message: Update XSensModelStyle_URDFtemplate.urdf

File: Experiments/23links_human/templates/XSensModelStyle_URDFtemplate.urdf (robot description, URDF)
Before this commit: robot XSensStyleModel_template, 67 links, 66 joints
Links:
- link Head_f1: mass 0 0 0 -> FAKEMASS; geometry 
- link Head_f2: mass 0 0 0 -> FAKEMASS; geometry 
- link L3_f1: mass 0 0 0 -> FAKEMASS; geometry 
- link L3_f2: mass 0 0 0 -> FAKEMASS; geometry 
- link L5_f1: mass 0 0 0 -> FAKEMASS; geometry 
- link L5_f2: mass 0 0 0 -> FAKEMASS; geometry 
- link LeftFoot_f1: mass 0 0 0 -> FAKEMASS; geometry 
- link LeftFoot_f2: mass 0 0 0 -> FAKEMASS; geometry 
- link LeftForeArm_f1: mass 0 0 0 -> FAKEMASS; geometry 
- link LeftForeArm_f2: mass 0 0 0 -> FAKEMASS; geometry 
- link LeftHand_f1: mass 0 0 0 -> FAKEMASS; geometry 
- link LeftHand_f2: mass 0 0 0 -> FAKEMASS; geometry 
- link LeftLowerLeg_f1: mass 0 0 0 -> FAKEMASS; geometry 
- link LeftLowerLeg_f2: mass 0 0 0 -> FAKEMASS; geometry 
- link LeftShoulder_f1: mass 0 0 0 -> FAKEMASS; geometry 
- link LeftShoulder_f2: mass 0 0 0 -> FAKEMASS; geometry 
- link LeftToe_f1: mass 0 0 0 -> FAKEMASS; geometry 
- link LeftToe_f2: mass 0 0 0 -> FAKEMASS; geometry 
- link LeftUpperArm_f1: mass 0 0 0 -> FAKEMASS; geometry 
- link LeftUpperArm_f2: mass 0 0 0 -> FAKEMASS; geometry 
- link LeftUpperLeg_f1: mass 0 0 0 -> FAKEMASS; geometry 
- link LeftUpperLeg_f2: mass 0 0 0 -> FAKEMASS; geometry 
- link Neck_f1: mass 0 0 0 -> FAKEMASS; geometry 
- link Neck_f2: mass 0 0 0 -> FAKEMASS; geometry 
- link RightFoot_f1: mass 0 0 0 -> FAKEMASS; geometry 
- link RightFoot_f2: mass 0 0 0 -> FAKEMASS; geometry 
- link RightForeArm_f1: mass 0 0 0 -> FAKEMASS; geometry 
- link RightForeArm_f2: mass 0 0 0 -> FAKEMASS; geometry 
- link RightHand_f1: mass 0 0 0 -> FAKEMASS; geometry 
- link RightHand_f2: mass 0 0 0 -> FAKEMASS; geometry 
- link RightLowerLeg_f1: mass 0 0 0 -> FAKEMASS; geometry 
- link RightLowerLeg_f2: mass 0 0 0 -> FAKEMASS; geometry 
- link RightShoulder_f1: mass 0 0 0 -> FAKEMASS; geometry 
- link RightShoulder_f2: mass 0 0 0 -> FAKEMASS; geometry 
- link RightToe_f1: mass 0 0 0 -> FAKEMASS; geometry 
- link RightToe_f2: mass 0 0 0 -> FAKEMASS; geometry 
- link RightUpperArm_f1: mass 0 0 0 -> FAKEMASS; geometry 
- link RightUpperArm_f2: mass 0 0 0 -> FAKEMASS; geometry 
- link RightUpperLeg_f1: mass 0 0 0 -> FAKEMASS; geometry 
- link RightUpperLeg_f2: mass 0 0 0 -> FAKEMASS; geometry 
- link T12_f1: mass 0 0 0 -> FAKEMASS; geometry 
- link T12_f2: mass 0 0 0 -> FAKEMASS; geometry 
- link T8_f1: mass 0 0 0 -> FAKEMASS; geometry 
- link T8_f2: mass 0 0 0 -> FAKEMASS; geometry 

Commit message: minor modifications/fixed typos on models

File: Experiments/23links_human/templates/XSensModelStyle_URDFtemplate.urdf (robot description, URDF)
Before this commit: robot XSensStyleModel_template, 67 links, 66 joints
Joints:
- joint jC1Head_rotx: limit lower=-10.0 effort=30 velocity=1.0 -> lower=-10.0 upper=10.0 effort=30 velocity=1.0
- joint jC1Head_roty: limit lower=-10.0 effort=30 velocity=1.0 -> lower=-10.0 upper=10.0 effort=30 velocity=1.0
- joint jC1Head_rotz: limit lower=-10.0 effort=30 velocity=1.0 -> lower=-10.0 upper=10.0 effort=30 velocity=1.0
- joint jL1T12_rotx: limit lower=-10.0 effort=30 velocity=1.0 -> lower=-10.0 upper=10.0 effort=30 velocity=1.0
- joint jL1T12_roty: limit lower=-10.0 effort=30 velocity=1.0 -> lower=-10.0 upper=10.0 effort=30 velocity=1.0
- joint jL1T12_rotz: limit lower=-10.0 effort=30 velocity=1.0 -> lower=-10.0 upper=10.0 effort=30 velocity=1.0
- joint jL4L3_rotx: limit lower=-10.0 effort=30 velocity=1.0 -> lower=-10.0 upper=10.0 effort=30 velocity=1.0
- joint jL4L3_roty: limit lower=-10.0 effort=30 velocity=1.0 -> lower=-10.0 upper=10.0 effort=30 velocity=1.0
- joint jL4L3_rotz: limit lower=-10.0 effort=30 velocity=1.0 -> lower=-10.0 upper=10.0 effort=30 velocity=1.0
- joint jL5S1_rotx: limit lower=-10.0 effort=30 velocity=1.0 -> lower=-10.0 upper=10.0 effort=30 velocity=1.0
- joint jL5S1_roty: limit lower=-10.0 effort=30 velocity=1.0 -> lower=-10.0 upper=10.0 effort=30 velocity=1.0
- joint jL5S1_rotz: limit lower=-10.0 effort=30 velocity=1.0 -> lower=-10.0 upper=10.0 effort=30 velocity=1.0
- joint jLeftAnkle_rotx: limit lower=-10.0 effort=30 velocity=1.0 -> lower=-10.0 upper=10.0 effort=30 velocity=1.0
- joint jLeftAnkle_roty: limit lower=-10.0 effort=30 velocity=1.0 -> lower=-10.0 upper=10.0 effort=30 velocity=1.0
- joint jLeftAnkle_rotz: limit lower=-10.0 effort=30 velocity=1.0 -> lower=-10.0 upper=10.0 effort=30 velocity=1.0
- joint jLeftBallFoot_rotx: limit lower=-10.0 effort=30 velocity=1.0 -> lower=-10.0 upper=10.0 effort=30 velocity=1.0
- joint jLeftBallFoot_roty: limit lower=-10.0 effort=30 velocity=1.0 -> lower=-10.0 upper=10.0 effort=30 velocity=1.0
- joint jLeftBallFoot_rotz: limit lower=-10.0 effort=30 velocity=1.0 -> lower=-10.0 upper=10.0 effort=30 velocity=1.0
- joint jLeftC7Shoulder_rotx: limit lower=-10.0 effort=30 velocity=1.0 -> lower=-10.0 upper=10.0 effort=30 velocity=1.0
- joint jLeftC7Shoulder_roty: limit lower=-10.0 effort=30 velocity=1.0 -> lower=-10.0 upper=10.0 effort=30 velocity=1.0
- joint jLeftC7Shoulder_rotz: limit lower=-10.0 effort=30 velocity=1.0 -> lower=-10.0 upper=10.0 effort=30 velocity=1.0
- joint jLeftElbow_rotx: limit lower=-10.0 effort=30 velocity=1.0 -> lower=-10.0 upper=10.0 effort=30 velocity=1.0
- joint jLeftElbow_roty: limit lower=-10.0 effort=30 velocity=1.0 -> lower=-10.0 upper=10.0 effort=30 velocity=1.0
- joint jLeftElbow_rotz: limit lower=-10.0 effort=30 velocity=1.0 -> lower=-10.0 upper=10.0 effort=30 velocity=1.0
- joint jLeftHip_rotx: limit lower=-10.0 effort=30 velocity=1.0 -> lower=-10.0 upper=10.0 effort=30 velocity=1.0
- joint jLeftHip_roty: limit lower=-10.0 effort=30 velocity=1.0 -> lower=-10.0 upper=10.0 effort=30 velocity=1.0
- joint jLeftHip_rotz: limit lower=-10.0 effort=30 velocity=1.0 -> lower=-10.0 upper=10.0 effort=30 velocity=1.0
- joint jLeftKnee_rotx: limit lower=-10.0 effort=30 velocity=1.0 -> lower=-10.0 upper=10.0 effort=30 velocity=1.0
- joint jLeftKnee_roty: limit lower=-10.0 effort=30 velocity=1.0 -> lower=-10.0 upper=10.0 effort=30 velocity=1.0
- joint jLeftKnee_rotz: limit lower=-10.0 effort=30 velocity=1.0 -> lower=-10.0 upper=10.0 effort=30 velocity=1.0
- joint jLeftWrist_rotx: limit lower=-10.0 effort=30 velocity=1.0 -> lower=-10.0 upper=10.0 effort=30 velocity=1.0
- joint jLeftWrist_roty: limit lower=-10.0 effort=30 velocity=1.0 -> lower=-10.0 upper=10.0 effort=30 velocity=1.0
- joint jLeftWrist_rotz: limit lower=-10.0 effort=30 velocity=1.0 -> lower=-10.0 upper=10.0 effort=30 velocity=1.0
- joint jRightAnkle_rotx: limit lower=-10.0 effort=30 velocity=1.0 -> lower=-10.0 upper=10.0 effort=30 velocity=1.0
- joint jRightAnkle_roty: limit lower=-10.0 effort=30 velocity=1.0 -> lower=-10.0 upper=10.0 effort=30 velocity=1.0
- joint jRightAnkle_rotz: limit lower=-10.0 effort=30 velocity=1.0 -> lower=-10.0 upper=10.0 effort=30 velocity=1.0
- joint jRightBallFoot_rotx: limit lower=-10.0 effort=30 velocity=1.0 -> lower=-10.0 upper=10.0 effort=30 velocity=1.0
- joint jRightBallFoot_roty: limit lower=-10.0 effort=30 velocity=1.0 -> lower=-10.0 upper=10.0 effort=30 velocity=1.0
- joint jRightBallFoot_rotz: limit lower=-10.0 effort=30 velocity=1.0 -> lower=-10.0 upper=10.0 effort=30 velocity=1.0
- joint jRightC7Shoulder_rotx: limit lower=-10.0 effort=30 velocity=1.0 -> lower=-10.0 upper=10.0 effort=30 velocity=1.0
- joint jRightC7Shoulder_roty: limit lower=-10.0 effort=30 velocity=1.0 -> lower=-10.0 upper=10.0 effort=30 velocity=1.0
- joint jRightC7Shoulder_rotz: limit lower=-10.0 effort=30 velocity=1.0 -> lower=-10.0 upper=10.0 effort=30 velocity=1.0
- joint jRightElbow_rotx: limit lower=-10.0 effort=30 velocity=1.0 -> lower=-10.0 upper=10.0 effort=30 velocity=1.0
- joint jRightElbow_roty: limit lower=-10.0 effort=30 velocity=1.0 -> lower=-10.0 upper=10.0 effort=30 velocity=1.0
- joint jRightElbow_rotz: limit lower=-10.0 effort=30 velocity=1.0 -> lower=-10.0 upper=10.0 effort=30 velocity=1.0
- joint jRightHip_rotx: limit lower=-10.0 effort=30 velocity=1.0 -> lower=-10.0 upper=10.0 effort=30 velocity=1.0
- joint jRightHip_roty: limit lower=-10.0 effort=30 velocity=1.0 -> lower=-10.0 upper=10.0 effort=30 velocity=1.0
- joint jRightHip_rotz: limit lower=-10.0 effort=30 velocity=1.0 -> lower=-10.0 upper=10.0 effort=30 velocity=1.0
- joint jRightKnee_rotx: limit lower=-10.0 effort=30 velocity=1.0 -> lower=-10.0 upper=10.0 effort=30 velocity=1.0
- joint jRightKnee_roty: limit lower=-10.0 effort=30 velocity=1.0 -> lower=-10.0 upper=10.0 effort=30 velocity=1.0
- joint jRightKnee_rotz: limit lower=-10.0 effort=30 velocity=1.0 -> lower=-10.0 upper=10.0 effort=30 velocity=1.0
- joint jRightWrist_rotx: limit lower=-10.0 effort=30 velocity=1.0 -> lower=-10.0 upper=10.0 effort=30 velocity=1.0
- joint jRightWrist_roty: limit lower=-10.0 effort=30 velocity=1.0 -> lower=-10.0 upper=10.0 effort=30 velocity=1.0
- joint jRightWrist_rotz: limit lower=-10.0 effort=30 velocity=1.0 -> lower=-10.0 upper=10.0 effort=30 velocity=1.0
- joint jT1C7_rotx: limit lower=-10.0 effort=30 velocity=1.0 -> lower=-10.0 upper=10.0 effort=30 velocity=1.0
- joint jT1C7_roty: limit lower=-10.0 effort=30 velocity=1.0 -> lower=-10.0 upper=10.0 effort=30 velocity=1.0
- joint jT1C7_rotz: limit lower=-10.0 effort=30 velocity=1.0 -> lower=-10.0 upper=10.0 effort=30 velocity=1.0
- joint jT9T8_rotx: limit lower=-10.0 effort=30 velocity=1.0 -> lower=-10.0 upper=10.0 effort=30 velocity=1.0
- joint jT9T8_roty: limit lower=-10.0 effort=30 velocity=1.0 -> lower=-10.0 upper=10.0 effort=30 velocity=1.0
- joint jT9T8_rotz: limit lower=-10.0 effort=30 velocity=1.0 -> lower=-10.0 upper=10.0 effort=30 velocity=1.0

Commit message: added model templates with 48 DOFs

File: Experiments/23links_human/templates/XSensModelStyle_URDFtemplate.urdf (robot description, URDF)
Before this commit: robot XSensStyleModel_template, 67 links, 66 joints
Links:
- removed link Head_f2
- removed link L3_f2
- removed link L5_f2
- removed link LeftForeArm_f2
- removed link LeftHand_f2
- removed link LeftLowerLeg_f2
- removed link LeftShoulder_f1
- removed link LeftShoulder_f2
- removed link LeftToe_f1
- removed link LeftToe_f2
- removed link RightForeArm_f2
- removed link RightHand_f2
- removed link RightLowerLeg_f2
- removed link RightShoulder_f1
- removed link RightShoulder_f2
- removed link RightToe_f1
- removed link RightToe_f2
- removed link T12_f2
Joints:
- removed joint jC1Head_rotz
- removed joint jL1T12_rotz
- removed joint jL4L3_rotz
- removed joint jL5S1_rotz
- removed joint jLeftBallFoot_rotx
- removed joint jLeftBallFoot_rotz
- removed joint jLeftC7Shoulder_roty
- removed joint jLeftC7Shoulder_rotz
- removed joint jLeftElbow_rotx
- removed joint jLeftKnee_rotx
- removed joint jLeftWrist_roty
- removed joint jRightBallFoot_rotx
- removed joint jRightBallFoot_rotz
- removed joint jRightC7Shoulder_roty
- removed joint jRightC7Shoulder_rotz
- removed joint jRightElbow_rotx
- removed joint jRightKnee_rotx
- removed joint jRightWrist_roty
- joint jC1Head_rotx: limit lower=-10.0 upper=10.0 effort=30 velocity=1.0 -> lower=-0.610865 upper=0.610865 effort=30 velocity=1.0
- joint jC1Head_roty: child Head_f2 -> Head; limit lower=-10.0 upper=10.0 effort=30 velocity=1.0 -> lower=-0.436332 upper=0.174533 effort=30 velocity=1.0
- joint jL1T12_rotx: limit lower=-10.0 upper=10.0 effort=30 velocity=1.0 -> lower=-0.610865 upper=0.610865 effort=30 velocity=1.0
- joint jL1T12_roty: child T12_f2 -> T12; limit lower=-10.0 upper=10.0 effort=30 velocity=1.0 -> lower=-0.523599 upper=1.309 effort=30 velocity=1.0
- joint jL4L3_rotx: limit lower=-10.0 upper=10.0 effort=30 velocity=1.0 -> lower=-0.610865 upper=0.610865 effort=30 velocity=1.0
- joint jL4L3_roty: child L3_f2 -> L3; limit lower=-10.0 upper=10.0 effort=30 velocity=1.0 -> lower=-0.523599 upper=1.309 effort=30 velocity=1.0
- joint jL5S1_rotx: limit lower=-10.0 upper=10.0 effort=30 velocity=1.0 -> lower=-0.610865 upper=0.610865 effort=30 velocity=1.0
- joint jL5S1_roty: child L5_f2 -> L5; limit lower=-10.0 upper=10.0 effort=30 velocity=1.0 -> lower=-0.523599 upper=1.309 effort=30 velocity=1.0
- joint jLeftAnkle_rotx: limit lower=-10.0 upper=10.0 effort=30 velocity=1.0 -> lower=-0.610865 upper=0.785398 effort=30 velocity=1.0
- joint jLeftAnkle_roty: limit lower=-10.0 upper=10.0 effort=30 velocity=1.0 -> lower=-0.523599 upper=0.872665 effort=30 velocity=1.0
- joint jLeftAnkle_rotz: limit lower=-10.0 upper=10.0 effort=30 velocity=1.0 -> lower=-0.872665 upper=0.436332 effort=30 velocity=1.0
- joint jLeftBallFoot_roty: child LeftToe_f2 -> LeftToe; limit lower=-10.0 upper=10.0 effort=30 velocity=1.0 -> lower=-0.174533 upper=1.5708 effort=30 velocity=1.0; origin xyz=0 0 0 rpy=0 0 0 -> xyz=jLeftBallFoot_ORIGIN rpy=0 0 0; parent LeftToe_f1 -> LeftFoot
- joint jLeftC7Shoulder_rotx: child LeftShoulder_f1 -> LeftShoulder; limit lower=-10.0 upper=10.0 effort=30 velocity=1.0 -> lower=-0.0872665 upper=0.785398 effort=30 velocity=1.0
- joint jLeftElbow_roty: child LeftForeArm_f2 -> LeftForeArm_f1; limit lower=-10.0 upper=10.0 effort=30 velocity=1.0 -> lower=-1.5708 upper=1.48353 effort=30 velocity=1.0; origin xyz=0 0 0 rpy=0 0 0 -> xyz=jLeftElbow_ORIGIN rpy=0 0 0; parent LeftForeArm_f1 -> LeftUpperArm
- joint jLeftElbow_rotz: limit lower=-10.0 upper=10.0 effort=30 velocity=1.0 -> lower=-2.53073 upper=0 effort=30 velocity=1.0; parent LeftForeArm_f2 -> LeftForeArm_f1
- joint jLeftHip_rotx: limit lower=-10.0 upper=10.0 effort=30 velocity=1.0 -> lower=-0.523599 upper=0.785398 effort=30 velocity=1.0
- joint jLeftHip_roty: limit lower=-10.0 upper=10.0 effort=30 velocity=1.0 -> lower=-0.261799 upper=2.0944 effort=30 velocity=1.0
- joint jLeftHip_rotz: limit lower=-10.0 upper=10.0 effort=30 velocity=1.0 -> lower=-0.785398 upper=0.785398 effort=30 velocity=1.0
- joint jLeftKnee_roty: child LeftLowerLeg_f2 -> LeftLowerLeg_f1; limit lower=-10.0 upper=10.0 effort=30 velocity=1.0 -> lower=0 upper=2.35619 effort=30 velocity=1.0; origin xyz=0 0 0 rpy=0 0 0 -> xyz=jLeftKnee_ORIGIN rpy=0 0 0; parent LeftLowerLeg_f1 -> LeftUpperLeg
- joint jLeftKnee_rotz: limit lower=-10.0 upper=10.0 effort=30 velocity=1.0 -> lower=-0.523599 upper=0.698132 effort=30 velocity=1.0; parent LeftLowerLeg_f2 -> LeftLowerLeg_f1
- joint jLeftShoulder_rotx: limit lower=-10.0 upper=10.0 effort=30 velocity=1.0 -> lower=-1.5708 upper=2.35619 effort=30 velocity=1.0
- joint jLeftShoulder_roty: limit lower=-10.0 upper=10.0 effort=30 velocity=1.0 -> lower=-1.5708 upper=1.5708 effort=30 velocity=1.0
- joint jLeftShoulder_rotz: limit lower=-10.0 upper=10.0 effort=30 velocity=1.0 -> lower=-3.14159 upper=0.785398 effort=30 velocity=1.0
- joint jLeftWrist_rotx: limit lower=-10.0 upper=10.0 effort=30 velocity=1.0 -> lower=-1.0472 upper=0.872665 effort=30 velocity=1.0
- joint jLeftWrist_rotz: limit lower=-10.0 upper=10.0 effort=30 velocity=1.0 -> lower=-0.349066 upper=0.523599 effort=30 velocity=1.0; parent LeftHand_f2 -> LeftHand_f1
- joint jRightAnkle_rotx: limit lower=-10.0 upper=10.0 effort=30 velocity=1.0 -> lower=-0.610865 upper=0.785398 effort=30 velocity=1.0
- joint jRightAnkle_roty: limit lower=-10.0 upper=10.0 effort=30 velocity=1.0 -> lower=-0.523599 upper=0.872665 effort=30 velocity=1.0
- joint jRightAnkle_rotz: limit lower=-10.0 upper=10.0 effort=30 velocity=1.0 -> lower=-0.436332 upper=0.872665 effort=30 velocity=1.0
- joint jRightBallFoot_roty: child RightToe_f2 -> RightToe; limit lower=-10.0 upper=10.0 effort=30 velocity=1.0 -> lower=-0.174533 upper=1.5708 effort=30 velocity=1.0; origin xyz=0 0 0 rpy=0 0 0 -> xyz=jRightBallFoot_ORIGIN rpy=0 0 0; parent RightToe_f1 -> RightFoot
- joint jRightC7Shoulder_rotx: child RightShoulder_f1 -> RightShoulder; limit lower=-10.0 upper=10.0 effort=30 velocity=1.0 -> lower=-0.0872665 upper=0.785398 effort=30 velocity=1.0
- joint jRightElbow_roty: child RightForeArm_f2 -> RightForeArm_f1; limit lower=-10.0 upper=10.0 effort=30 velocity=1.0 -> lower=-1.5708 upper=1.48353 effort=30 velocity=1.0; origin xyz=0 0 0 rpy=0 0 0 -> xyz=jRightElbow_ORIGIN rpy=0 0 0; parent RightForeArm_f1 -> RightUpperArm
- joint jRightElbow_rotz: limit lower=-10.0 upper=10.0 effort=30 velocity=1.0 -> lower=0 upper=2.53073 effort=30 velocity=1.0; parent RightForeArm_f2 -> RightForeArm_f1
- joint jRightHip_rotx: limit lower=-10.0 upper=10.0 effort=30 velocity=1.0 -> lower=-0.523599 upper=0.785398 effort=30 velocity=1.0
- joint jRightHip_roty: limit lower=-10.0 upper=10.0 effort=30 velocity=1.0 -> lower=-0.261799 upper=2.0944 effort=30 velocity=1.0
- joint jRightHip_rotz: limit lower=-10.0 upper=10.0 effort=30 velocity=1.0 -> lower=-0.785398 upper=0.785398 effort=30 velocity=1.0
- joint jRightKnee_roty: child RightLowerLeg_f2 -> RightLowerLeg_f1; limit lower=-10.0 upper=10.0 effort=30 velocity=1.0 -> lower=0 upper=2.35619 effort=30 velocity=1.0; origin xyz=0 0 0 rpy=0 0 0 -> xyz=jRightKnee_ORIGIN rpy=0 0 0; parent RightLowerLeg_f1 -> RightUpperLeg
- joint jRightKnee_rotz: limit lower=-10.0 upper=10.0 effort=30 velocity=1.0 -> lower=-0.698132 upper=0.523599 effort=30 velocity=1.0; parent RightLowerLeg_f2 -> RightLowerLeg_f1
- joint jRightShoulder_rotx: limit lower=-10.0 upper=10.0 effort=30 velocity=1.0 -> lower=-2.35619 upper=1.5708 effort=30 velocity=1.0
- joint jRightShoulder_roty: limit lower=-10.0 upper=10.0 effort=30 velocity=1.0 -> lower=-1.5708 upper=1.5708 effort=30 velocity=1.0
- joint jRightShoulder_rotz: limit lower=-10.0 upper=10.0 effort=30 velocity=1.0 -> lower=-0.785398 upper=3.14159 effort=30 velocity=1.0
- joint jRightWrist_rotx: limit lower=-10.0 upper=10.0 effort=30 velocity=1.0 -> lower=-0.872665 upper=1.0472 effort=30 velocity=1.0
- joint jRightWrist_rotz: limit lower=-10.0 upper=10.0 effort=30 velocity=1.0 -> lower=-0.523599 upper=0.349066 effort=30 velocity=1.0; parent RightHand_f2 -> RightHand_f1
- joint jT1C7_rotx: limit lower=-10.0 upper=10.0 effort=30 velocity=1.0 -> lower=-0.610865 upper=0.610865 effort=30 velocity=1.0
- joint jT1C7_roty: limit lower=-10.0 upper=10.0 effort=30 velocity=1.0 -> lower=-0.959931 upper=1.5708 effort=30 velocity=1.0
- joint jT1C7_rotz: limit lower=-10.0 upper=10.0 effort=30 velocity=1.0 -> lower=-1.22173 upper=1.22173 effort=30 velocity=1.0
- joint jT9T8_rotx: limit lower=-10.0 upper=10.0 effort=30 velocity=1.0 -> lower=-0.349066 upper=0.349066 effort=30 velocity=1.0
- joint jT9T8_roty: limit lower=-10.0 upper=10.0 effort=30 velocity=1.0 -> lower=-0.261799 upper=0.698132 effort=30 velocity=1.0
- joint jT9T8_rotz: limit lower=-10.0 upper=10.0 effort=30 velocity=1.0 -> lower=-0.610865 upper=0.610865 effort=30 velocity=1.0
